File: Buttons.sch (KiCad schematic (older format))
At the start: 7 parts, among them SW1 SW_PUSH, SW2 SW_PUSH, SW3 SW_PUSH, SW4 SW_PUSH, SW5 SW_PUSH, SW6 SW_PUSH, SW7 SW_PUSH

Commit message: v1.5 Finalized
Parts:
- SW1, SW2, SW3, SW4, SW5, SW6, SW7: LSCS (none) -> C221889
Changed lines of the file:
@@
 $Descr A4 11693 8268
 encoding utf-8
-Sheet 2 19
+Sheet 2 15
 Title ""
 Date ""
@@
 F 2 "Button_Switch_THT:SW_Tactile_SPST_Angled_PTS645Vx83-2LFS" H 2000 4700 60  0001 C CNN
 F 3 "" H 2000 4700 60  0000 C CNN
+F 4 "C221889" H 2000 4700 50  0001 C CNN "LSCS"
 	1    2000 4700
 	1    0    0    -1
@@
 F 2 "Button_Switch_THT:SW_Tactile_SPST_Angled_PTS645Vx83-2LFS" H 3450 4700 60  0001 C CNN
 F 3 "" H 3450 4700 60  0000 C CNN
+F 4 "C221889" H 3450 4700 50  0001 C CNN "LSCS"
 	1    3450 4700
 	1    0    0    -1
@@
 F 2 "Button_Switch_THT:SW_Tactile_SPST_Angled_PTS645Vx83-2LFS" H 4850 4700 60  0001 C CNN
 F 3 "" H 4850 4700 60  0000 C CNN
+F 4 "C221889" H 4850 4700 50  0001 C CNN "LSCS"
 	1    4850 4700
 	1    0    0    -1
@@
 P 2350 4700
 AR Path="/6149D0E7" Ref="#PWR?"  Part="1"
-AR Path="/614940F6/6149D0E7" Ref="#PWR06"  Part="1"
-F 0 "#PWR06" H 2350 4450 50  0001 C CNN
+AR Path="/614940F6/6149D0E7" Ref="#PWR016"  Part="1"
+F 0 "#PWR016" H 2350 4450 50  0001 C CNN
 F 1 "GND" V 2355 4572 50  0000 R CNN
 F 2 "" H 2350 4700 50  0001 C CNN
@@
 P 3800 4700
 AR Path="/6149D0ED" Ref="#PWR?"  Part="1"
-AR Path="/614940F6/6149D0ED" Ref="#PWR09"  Part="1"
-F 0 "#PWR09" H 3800 4450 50  0001 C CNN
+AR Path="/614940F6/6149D0ED" Ref="#PWR019"  Part="1"
+F 0 "#PWR019" H 3800 4450 50  0001 C CNN
 F 1 "GND" V 3805 4572 50  0000 R CNN
 F 2 "" H 3800 4700 50  0001 C CNN
@@
 P 5200 4700
 AR Path="/6149D0F3" Ref="#PWR?"  Part="1"
-AR Path="/614940F6/6149D0F3" Ref="#PWR011"  Part="1"
-F 0 "#PWR011" H 5200 4450 50  0001 C CNN
+AR Path="/614940F6/6149D0F3" Ref="#PWR021"  Part="1"
+F 0 "#PWR021" H 5200 4450 50  0001 C CNN
 F 1 "GND" V 5205 4572 50  0000 R CNN
 F 2 "" H 5200 4700 50  0001 C CNN
@@
 F 2 "Button_Switch_THT:SW_Tactile_SPST_Angled_PTS645Vx83-2LFS" H 2000 5100 60  0001 C CNN
 F 3 "" H 2000 5100 60  0000 C CNN
+F 4 "C221889" H 2000 5100 50  0001 C CNN "LSCS"
 	1    2000 5100
 	1    0    0    -1
@@
 F 2 "Button_Switch_THT:SW_Tactile_SPST_Angled_PTS645Vx83-2LFS" H 3450 5100 60  0001 C CNN
 F 3 "" H 3450 5100 60  0000 C CNN
+F 4 "C221889" H 3450 5100 50  0001 C CNN "LSCS"
 	1    3450 5100
 	1    0    0    -1
@@
 F 2 "Button_Switch_THT:SW_Tactile_SPST_Angled_PTS645Vx83-2LFS" H 4850 5100 60  0001 C CNN
 F 3 "" H 4850 5100 60  0000 C CNN
+F 4 "C221889" H 4850 5100 50  0001 C CNN "LSCS"
 	1    4850 5100
 	1    0    0    -1
@@
 P 2350 5100
 AR Path="/6149D114" Ref="#PWR?"  Part="1"
-AR Path="/614940F6/6149D114" Ref="#PWR07"  Part="1"
-F 0 "#PWR07" H 2350 4850 50  0001 C CNN
+AR Path="/614940F6/6149D114" Ref="#PWR017"  Part="1"
+F 0 "#PWR017" H 2350 4850 50  0001 C CNN
 F 1 "GND" V 2355 4972 50  0000 R CNN
 F 2 "" H 2350 5100 50  0001 C CNN
@@
 P 3800 5100
 AR Path="/6149D11A" Ref="#PWR?"  Part="1"
-AR Path="/614940F6/6149D11A" Ref="#PWR010"  Part="1"
-F 0 "#PWR010" H 3800 4850 50  0001 C CNN
+AR Path="/614940F6/6149D11A" Ref="#PWR020"  Part="1"
+F 0 "#PWR020" H 3800 4850 50  0001 C CNN
 F 1 "GND" V 3805 4972 50  0000 R CNN
 F 2 "" H 3800 5100 50  0001 C CNN
@@
 P 5200 5100
 AR Path="/6149D120" Ref="#PWR?"  Part="1"
-AR Path="/614940F6/6149D120" Ref="#PWR012"  Part="1"
-F 0 "#PWR012" H 5200 4850 50  0001 C CNN
+AR Path="/614940F6/6149D120" Ref="#PWR022"  Part="1"
+F 0 "#PWR022" H 5200 4850 50  0001 C CNN
 F 1 "GND" V 5205 4972 50  0000 R CNN
 F 2 "" H 5200 5100 50  0001 C CNN
@@
 F 2 "Button_Switch_THT:SW_Tactile_SPST_Angled_PTS645Vx83-2LFS" H 2000 5500 60  0001 C CNN
 F 3 "" H 2000 5500 60  0000 C CNN
+F 4 "C221889" H 2000 5500 50  0001 C CNN "LSCS"
 	1    2000 5500
 	1    0    0    -1
@@
 P 2350 5500
 AR Path="/616BA3E1" Ref="#PWR?"  Part="1"
-AR Path="/614940F6/616BA3E1" Ref="#PWR08"  Part="1"
-F 0 "#PWR08" H 2350 5250 50  0001 C CNN
+AR Path="/614940F6/616BA3E1" Ref="#PWR018"  Part="1"
+F 0 "#PWR018" H 2350 5250 50  0001 C CNN
 F 1 "GND" V 2355 5372 50  0000 R CNN
 F 2 "" H 2350 5500 50  0001 C CNN
