File: Crystal.sch (KiCad schematic (older format))
At the start: 4 parts, among them Y1 ABLS-12.000MHZ-B4-T

Commit message: v1.5 Finalized
Parts:
- C15, C16: footprint Capacitor_SMD:C_0402_1005Metric -> Capacitor_SMD:C_0805_2012Metric; LSCS (none) -> C1557
- R3: footprint Capacitor_SMD:C_0402_1005Metric -> Resistor_SMD:R_0805_2012Metric; LSCS (none) -> C11702
- Y1: LSCS (none) -> C596818
Changed lines of the file:
@@
 F 0 "C15" H 4865 3696 50  0000 L CNN
 F 1 "27p" H 4865 3605 50  0000 L CNN
-F 2 "Capacitor_SMD:C_0402_1005Metric" H 4788 3500 50  0001 C CNN
+F 2 "Capacitor_SMD:C_0805_2012Metric" H 4788 3500 50  0001 C CNN
 F 3 "~" H 4750 3650 50  0001 C CNN
+F 4 "C1557" H 4750 3650 50  0001 C CNN "LSCS"
 	1    4750 3650
 	0    1    1    0
@@
 F 0 "C16" H 4865 4096 50  0000 L CNN
 F 1 "27p" H 4865 4005 50  0000 L CNN
-F 2 "Capacitor_SMD:C_0402_1005Metric" H 4788 3900 50  0001 C CNN
+F 2 "Capacitor_SMD:C_0805_2012Metric" H 4788 3900 50  0001 C CNN
 F 3 "~" H 4750 4050 50  0001 C CNN
+F 4 "C1557" H 4750 4050 50  0001 C CNN "LSCS"
 	1    4750 4050
 	0    1    1    0
@@
 F 0 "R3" V 5843 4050 50  0000 C CNN
 F 1 "1k" V 5934 4050 50  0000 C CNN
-F 2 "Capacitor_SMD:C_0402_1005Metric" V 5980 4050 50  0001 C CNN
+F 2 "Resistor_SMD:R_0805_2012Metric" V 5980 4050 50  0001 C CNN
 F 3 "~" H 6050 4050 50  0001 C CNN
+F 4 "C11702" H 6050 4050 50  0001 C CNN "LSCS"
 	1    6050 4050
 	0    1    1    0
@@
 F 2 "RP2040_minimal:Crystal_SMD_HC49-US" H 5350 3850 50  0001 C CNN
 F 3 "~" H 5350 3850 50  0001 C CNN
+F 4 "C596818" H 5350 3850 50  0001 C CNN "LSCS"
 	1    5350 3850
 	0    1    1    0
