File: Flash.sch (KiCad schematic (older format))
At the start: 5 parts, among them SW8 SW_Push, U3 W25Q128JVS

Commit message: v1.5 Finalized
Parts:
- C17: footprint Capacitor_SMD:C_0402_1005Metric -> Capacitor_SMD:C_0805_2012Metric; LSCS (none) -> C60474
- R4: footprint Capacitor_SMD:C_0402_1005Metric -> Resistor_SMD:R_0805_2012Metric; LSCS (none) -> C11702
- R5: footprint Capacitor_SMD:C_0402_1005Metric -> Resistor_SMD:R_0805_2012Metric
- SW8: LSCS (none) -> C221762
- U3: LSCS (none) -> C97521
Changed lines of the file:
@@
 F 0 "C17" H 6565 3196 50  0000 L CNN
 F 1 "100n" H 6565 3105 50  0000 L CNN
-F 2 "Capacitor_SMD:C_0402_1005Metric" H 6488 3000 50  0001 C CNN
+F 2 "Capacitor_SMD:C_0805_2012Metric" H 6488 3000 50  0001 C CNN
 F 3 "~" H 6450 3150 50  0001 C CNN
+F 4 "C60474" H 6450 3150 50  0001 C CNN "LSCS"
 	1    6450 3150
 	1    0    0    -1
@@
 F 0 "R5" H 5670 3346 50  0000 L CNN
 F 1 "DNF" H 5670 3255 50  0000 L CNN
-F 2 "Capacitor_SMD:C_0402_1005Metric" V 5530 3300 50  0001 C CNN
+F 2 "Resistor_SMD:R_0805_2012Metric" V 5530 3300 50  0001 C CNN
 F 3 "~" H 5600 3300 50  0001 C CNN
 	1    5600 3300
@@
 F 2 "Package_SO:SOIC-8_5.23x5.23mm_P1.27mm" H 6200 4000 50  0001 C CNN
 F 3 "http://www.winbond.com/resource-files/w25q128jv_dtr%20revc%2003272018%20plus.pdf" H 6200 4000 50  0001 C CNN
+F 4 "C97521" H 6200 4000 50  0001 C CNN "LSCS"
 	1    6200 4000
 	1    0    0    -1
@@
 F 0 "R4" V 4793 3900 50  0000 C CNN
 F 1 "1k" V 4884 3900 50  0000 C CNN
-F 2 "Capacitor_SMD:C_0402_1005Metric" V 4930 3900 50  0001 C CNN
+F 2 "Resistor_SMD:R_0805_2012Metric" V 4930 3900 50  0001 C CNN
 F 3 "~" H 5000 3900 50  0001 C CNN
+F 4 "C11702" H 5000 3900 50  0001 C CNN "LSCS"
 	1    5000 3900
 	0    1    1    0
@@
 F 2 "Button_Switch_SMD:SW_Push_1P1T_NO_CK_KSC7xxJ" H 4150 4100 50  0001 C CNN
 F 3 "~" H 4150 4100 50  0001 C CNN
+F 4 "C221762" H 4150 3900 50  0001 C CNN "LSCS"
 	1    4150 3900
 	1    0    0    -1
