File: MCU.sch (KiCad schematic (older format))
At the start: 15 parts, among them J4 Debug, U1 RP2040

Commit message: v1.5 Finalized
Parts:
- C1, C10, C11, C2, C4, C6, C7, C8, C9: footprint Capacitor_SMD:C_0402_1005Metric -> Capacitor_SMD:C_0805_2012Metric; LSCS (none) -> C60474
- C3, C5: footprint Capacitor_SMD:C_0402_1005Metric -> Capacitor_SMD:C_0805_2012Metric; LSCS (none) -> C52923
- R1, R2: footprint Capacitor_SMD:C_0402_1005Metric -> Resistor_SMD:R_0805_2012Metric; LSCS (none) -> C25100
- U1: LSCS (none) -> C2040
Changed lines of the file:
@@
 F 2 "RP2040_minimal:RP2040-QFN-56" H 3300 5150 50  0001 C CNN
 F 3 "" H 3300 5150 50  0001 C CNN
+F 4 "C2040" H 4050 5150 50  0001 C CNN "LSCS"
 	1    4050 5150
 	1    0    0    -1
@@
 F 0 "R2" V 5693 3550 50  0000 C CNN
 F 1 "27" V 5784 3550 50  0000 C CNN
-F 2 "Capacitor_SMD:C_0402_1005Metric" V 5830 3550 50  0001 C CNN
+F 2 "Resistor_SMD:R_0805_2012Metric" V 5830 3550 50  0001 C CNN
 F 3 "~" H 5900 3550 50  0001 C CNN
+F 4 "C25100" H 5900 3550 50  0001 C CNN "LSCS"
 	1    5900 3550
 	0    1    1    0
@@
 F 0 "C4" H 5165 2096 50  0000 L CNN
 F 1 "100n" H 5165 2005 50  0000 L CNN
-F 2 "Capacitor_SMD:C_0402_1005Metric" H 5088 1900 50  0001 C CNN
+F 2 "Capacitor_SMD:C_0805_2012Metric" H 5088 1900 50  0001 C CNN
 F 3 "~" H 5050 2050 50  0001 C CNN
+F 4 "C60474" H 5050 2050 50  0001 C CNN "LSCS"
 	1    5050 2050
 	1    0    0    -1
@@
 F 0 "C6" H 5615 2096 50  0000 L CNN
 F 1 "100n" H 5615 2005 50  0000 L CNN
-F 2 "Capacitor_SMD:C_0402_1005Metric" H 5538 1900 50  0001 C CNN
+F 2 "Capacitor_SMD:C_0805_2012Metric" H 5538 1900 50  0001 C CNN
 F 3 "~" H 5500 2050 50  0001 C CNN
+F 4 "C60474" H 5500 2050 50  0001 C CNN "LSCS"
 	1    5500 2050
 	1    0    0    -1
@@
 F 0 "C7" H 6065 2096 50  0000 L CNN
 F 1 "100n" H 6065 2005 50  0000 L CNN
-F 2 "Capacitor_SMD:C_0402_1005Metric" H 5988 1900 50  0001 C CNN
+F 2 "Capacitor_SMD:C_0805_2012Metric" H 5988 1900 50  0001 C CNN
 F 3 "~" H 5950 2050 50  0001 C CNN
+F 4 "C60474" H 5950 2050 50  0001 C CNN "LSCS"
 	1    5950 2050
 	1    0    0    -1
@@
 F 0 "C8" H 6515 2096 50  0000 L CNN
 F 1 "100n" H 6515 2005 50  0000 L CNN
-F 2 "Capacitor_SMD:C_0402_1005Metric" H 6438 1900 50  0001 C CNN
+F 2 "Capacitor_SMD:C_0805_2012Metric" H 6438 1900 50  0001 C CNN
 F 3 "~" H 6400 2050 50  0001 C CNN
+F 4 "C60474" H 6400 2050 50  0001 C CNN "LSCS"
 	1    6400 2050
 	1    0    0    -1
@@
 F 0 "C9" H 6965 2096 50  0000 L CNN
 F 1 "100n" H 6965 2005 50  0000 L CNN
-F 2 "Capacitor_SMD:C_0402_1005Metric" H 6888 1900 50  0001 C CNN
+F 2 "Capacitor_SMD:C_0805_2012Metric" H 6888 1900 50  0001 C CNN
 F 3 "~" H 6850 2050 50  0001 C CNN
+F 4 "C60474" H 6850 2050 50  0001 C CNN "LSCS"
 	1    6850 2050
 	1    0    0    -1
@@
 F 0 "C10" H 7415 2096 50  0000 L CNN
 F 1 "100n" H 7415 2005 50  0000 L CNN
-F 2 "Capacitor_SMD:C_0402_1005Metric" H 7338 1900 50  0001 C CNN
+F 2 "Capacitor_SMD:C_0805_2012Metric" H 7338 1900 50  0001 C CNN
 F 3 "~" H 7300 2050 50  0001 C CNN
+F 4 "C60474" H 7300 2050 50  0001 C CNN "LSCS"
 	1    7300 2050
 	1    0    0    -1
@@
 F 0 "C11" H 7865 2096 50  0000 L CNN
 F 1 "100n" H 7865 2005 50  0000 L CNN
-F 2 "Capacitor_SMD:C_0402_1005Metric" H 7788 1900 50  0001 C CNN
+F 2 "Capacitor_SMD:C_0805_2012Metric" H 7788 1900 50  0001 C CNN
 F 3 "~" H 7750 2050 50  0001 C CNN
+F 4 "C60474" H 7750 2050 50  0001 C CNN "LSCS"
 	1    7750 2050
 	1    0    0    -1
@@
 F 0 "C1" H 2565 2096 50  0000 L CNN
 F 1 "100n" H 2565 2005 50  0000 L CNN
-F 2 "Capacitor_SMD:C_0402_1005Metric" H 2488 1900 50  0001 C CNN
+F 2 "Capacitor_SMD:C_0805_2012Metric" H 2488 1900 50  0001 C CNN
 F 3 "~" H 2450 2050 50  0001 C CNN
+F 4 "C60474" H 2450 2050 50  0001 C CNN "LSCS"
 	1    2450 2050
 	1    0    0    -1
@@
 F 0 "C2" H 3015 2096 50  0000 L CNN
 F 1 "100n" H 3015 2005 50  0000 L CNN
-F 2 "Capacitor_SMD:C_0402_1005Metric" H 2938 1900 50  0001 C CNN
+F 2 "Capacitor_SMD:C_0805_2012Metric" H 2938 1900 50  0001 C CNN
 F 3 "~" H 2900 2050 50  0001 C CNN
+F 4 "C60474" H 2900 2050 50  0001 C CNN "LSCS"
 	1    2900 2050
 	1    0    0    -1
@@
 F 0 "C3" H 3015 2696 50  0000 L CNN
 F 1 "1u" H 3015 2605 50  0000 L CNN
-F 2 "Capacitor_SMD:C_0402_1005Metric" H 2938 2500 50  0001 C CNN
+F 2 "Capacitor_SMD:C_0805_2012Metric" H 2938 2500 50  0001 C CNN
 F 3 "~" H 2900 2650 50  0001 C CNN
+F 4 "C52923" H 2900 2650 50  0001 C CNN "LSCS"
 	1    2900 2650
 	1    0    0    -1
@@
 F 0 "C5" H 5165 2696 50  0000 L CNN
 F 1 "1u" H 5165 2605 50  0000 L CNN
-F 2 "Capacitor_SMD:C_0402_1005Metric" H 5088 2500 50  0001 C CNN
+F 2 "Capacitor_SMD:C_0805_2012Metric" H 5088 2500 50  0001 C CNN
 F 3 "~" H 5050 2650 50  0001 C CNN
+F 4 "C52923" H 5050 2650 50  0001 C CNN "LSCS"
 	1    5050 2650
 	1    0    0    -1
@@
 F 0 "R1" V 5693 3250 50  0000 C CNN
 F 1 "27" V 5784 3250 50  0000 C CNN
-F 2 "Capacitor_SMD:C_0402_1005Metric" V 5830 3250 50  0001 C CNN
+F 2 "Resistor_SMD:R_0805_2012Metric" V 5830 3250 50  0001 C CNN
 F 3 "~" H 5900 3250 50  0001 C CNN
+F 4 "C25100" H 5900 3250 50  0001 C CNN "LSCS"
 	1    5900 3250
 	0    1    1    0
