File: OSFRD.sch (KiCad schematic (older format))
At the start: 2 parts, among them J1 20 Pin, J3 STEMMA QT

Commit message: v1.5 Finalized
Parts:
- added U1: Pico, MCU_RaspberryPi_and_Boards:RPi_Pico_SMD_TH, symbol MCU_RaspberryPi_and_Boards:Pico
- J1: footprint Connector_PinSocket_2.54mm:PinSocket_2x10_P2.54mm_Vertical -> Connector_PinSocket_2.54mm:PinSocket_2x10_P2.54mm_Vertical_SMD
- J2: renamed from J3; LSCS (none) -> C160404
Connections:
- net GPIO21 is gone; now on net GPIO14: J1.3 (Pin_3)
- net GPIO24 is gone; now on net GPIO3: J1.5 (Pin_5)
- net GPIO25 is gone; now on net GPIO0: J1.7 (Pin_7)
- net GPIO28_ADC2 is gone; now on net GPIO13: J1.8 (Pin_8)
- net +3V3: now also U1.36 (3V3)
- net +5V: now also U1.39 (VSYS)
- net GND: now also U1.13 (GND), U1.18 (GND), U1.23 (GND), U1.28 (GND), U1.3 (GND), U1.33 (AGND), U1.38 (GND), U1.8 (GND)
- net GPIO0: now also U1.1 (GPIO0); no longer J1.10 (Pin_10)
- net GPIO1: now also J1.4 (Pin_4), U1.2 (GPIO1)
- net GPIO13: now also U1.17 (GPIO13); no longer J1.16 (Pin_16)
- net GPIO14: now also U1.19 (GPIO14); no longer J1.15 (Pin_15)
- net GPIO16: now also J1.15 (Pin_15), U1.21 (GPIO16); no longer J1.1 (Pin_1)
- net GPIO17: now also U1.22 (GPIO17)
- net GPIO18: now also U1.24 (GPIO18)
- net GPIO19: now also J1.16 (Pin_16), U1.25 (GPIO19); no longer J1.4 (Pin_4)
- net GPIO20: now also J1.1 (Pin_1), U1.26 (GPIO20); no longer J1.2 (Pin_2)
- net GPIO26_I2C1_SDA: now also U1.31 (GPIO26_ADC0)
- net GPIO27_I2C1_SCL: now also U1.32 (GPIO27_ADC1)
- net GPIO3: now also U1.5 (GPIO3); no longer J1.11 (Pin_11)
- net GPIO5: now also U1.7 (GPIO5)
- net GPIO6: now also U1.9 (GPIO6)
- net GPIO7: now also U1.10 (GPIO7)
- net GPIO23 renamed GPIO4
- net GPIO4: now also U1.6 (GPIO4)
- net GPIO29_ADC3 renamed GPIO9
- net GPIO9: now also U1.12 (GPIO9)
- new net GPIO10: J1.10 (Pin_10), U1.14 (GPIO10)
- new net GPIO11: U1.15 (GPIO11)
- new net GPIO12: J1.11 (Pin_11), U1.16 (GPIO12)
- new net GPIO2: U1.4 (GPIO2)
- new net GPIO8: J1.2 (Pin_2), U1.11 (GPIO8)
- no-connect marks 8 -> 11
Other:
- moved on the sheet: J1, J2
