File: PlayerLEDs.sch (KiCad schematic (older format))
At the start: 8 parts

Commit message: v1.5 Finalized
Parts:
- U-CAP13, U-CAP14, U-CAP15, U-CAP16: footprint Capacitor_SMD:C_0805_2012Metric_Pad1.15x1.40mm_HandSolder -> Capacitor_SMD:C_0805_2012Metric; LSCS (none) -> C49678
Changed lines of the file:
@@
 $Descr A4 11693 8268
 encoding utf-8
-Sheet 15 19
+Sheet 15 15
 Title ""
 Date ""
@@
 F 0 "U-CAP13" V 2550 3500 50  0000 C CNN
 F 1 "0.1uF" V 2639 3350 50  0000 C CNN
-F 2 "Capacitor_SMD:C_0805_2012Metric_Pad1.15x1.40mm_HandSolder" H 2838 3200 50  0001 C CNN
+F 2 "Capacitor_SMD:C_0805_2012Metric" H 2838 3200 50  0001 C CNN
 F 3 "~" H 2800 3350 50  0001 C CNN
+F 4 "C49678" H 2800 3350 50  0001 C CNN "LSCS"
 	1    2800 3350
 	0    1    1    0
@@
 AR Path="/60DF69C3/6149FD9D" Ref="#PWR?"  Part="1"
 AR Path="/60DF76F4/6149FD9D" Ref="#PWR?"  Part="1"
-AR Path="/6149EA8A/6149FD9D" Ref="#PWR063"  Part="1"
-F 0 "#PWR063" H 3050 3100 50  0001 C CNN
+AR Path="/6149EA8A/6149FD9D" Ref="#PWR073"  Part="1"
+F 0 "#PWR073" H 3050 3100 50  0001 C CNN
 F 1 "GND" V 3055 3222 50  0000 R CNN
 F 2 "" H 3050 3350 50  0001 C CNN
@@
 AR Path="/60DF69C3/6149FDA4" Ref="#PWR?"  Part="1"
 AR Path="/60DF76F4/6149FDA4" Ref="#PWR?"  Part="1"
-AR Path="/6149EA8A/6149FDA4" Ref="#PWR062"  Part="1"
-F 0 "#PWR062" H 2500 4050 50  0001 C CNN
+AR Path="/6149EA8A/6149FDA4" Ref="#PWR072"  Part="1"
+F 0 "#PWR072" H 2500 4050 50  0001 C CNN
 F 1 "GND" V 2505 4172 50  0000 R CNN
 F 2 "" H 2500 4300 50  0001 C CNN
@@
 F 0 "U-CAP14" V 3350 3500 50  0000 C CNN
 F 1 "0.1uF" V 3439 3350 50  0000 C CNN
-F 2 "Capacitor_SMD:C_0805_2012Metric_Pad1.15x1.40mm_HandSolder" H 3638 3200 50  0001 C CNN
+F 2 "Capacitor_SMD:C_0805_2012Metric" H 3638 3200 50  0001 C CNN
 F 3 "~" H 3600 3350 50  0001 C CNN
+F 4 "C49678" H 3600 3350 50  0001 C CNN "LSCS"
 	1    3600 3350
 	0    1    1    0
@@
 AR Path="/60DF69C3/6149FDBB" Ref="#PWR?"  Part="1"
 AR Path="/60DF76F4/6149FDBB" Ref="#PWR?"  Part="1"
-AR Path="/6149EA8A/6149FDBB" Ref="#PWR066"  Part="1"
-F 0 "#PWR066" H 3850 3100 50  0001 C CNN
+AR Path="/6149EA8A/6149FDBB" Ref="#PWR076"  Part="1"
+F 0 "#PWR076" H 3850 3100 50  0001 C CNN
 F 1 "GND" V 3855 3222 50  0000 R CNN
 F 2 "" H 3850 3350 50  0001 C CNN
@@
 AR Path="/60DF69C3/6149FDC2" Ref="#PWR?"  Part="1"
 AR Path="/60DF76F4/6149FDC2" Ref="#PWR?"  Part="1"
-AR Path="/6149EA8A/6149FDC2" Ref="#PWR065"  Part="1"
-F 0 "#PWR065" H 3300 4050 50  0001 C CNN
+AR Path="/6149EA8A/6149FDC2" Ref="#PWR075"  Part="1"
+F 0 "#PWR075" H 3300 4050 50  0001 C CNN
 F 1 "GND" V 3305 4172 50  0000 R CNN
 F 2 "" H 3300 4300 50  0001 C CNN
@@
 F 0 "U-CAP15" V 4150 3500 50  0000 C CNN
 F 1 "0.1uF" V 4239 3350 50  0000 C CNN
-F 2 "Capacitor_SMD:C_0805_2012Metric_Pad1.15x1.40mm_HandSolder" H 4438 3200 50  0001 C CNN
+F 2 "Capacitor_SMD:C_0805_2012Metric" H 4438 3200 50  0001 C CNN
 F 3 "~" H 4400 3350 50  0001 C CNN
+F 4 "C49678" H 4400 3350 50  0001 C CNN "LSCS"
 	1    4400 3350
 	0    1    1    0
@@
 AR Path="/60DF69C3/6149FDD9" Ref="#PWR?"  Part="1"
 AR Path="/60DF76F4/6149FDD9" Ref="#PWR?"  Part="1"
-AR Path="/6149EA8A/6149FDD9" Ref="#PWR069"  Part="1"
-F 0 "#PWR069" H 4650 3100 50  0001 C CNN
+AR Path="/6149EA8A/6149FDD9" Ref="#PWR079"  Part="1"
+F 0 "#PWR079" H 4650 3100 50  0001 C CNN
 F 1 "GND" V 4655 3222 50  0000 R CNN
 F 2 "" H 4650 3350 50  0001 C CNN
@@
 AR Path="/60DF69C3/6149FDE0" Ref="#PWR?"  Part="1"
 AR Path="/60DF76F4/6149FDE0" Ref="#PWR?"  Part="1"
-AR Path="/6149EA8A/6149FDE0" Ref="#PWR068"  Part="1"
-F 0 "#PWR068" H 4100 4050 50  0001 C CNN
+AR Path="/6149EA8A/6149FDE0" Ref="#PWR078"  Part="1"
+F 0 "#PWR078" H 4100 4050 50  0001 C CNN
 F 1 "GND" V 4105 4172 50  0000 R CNN
 F 2 "" H 4100 4300 50  0001 C CNN
@@
 F 0 "U-CAP16" V 4950 3500 50  0000 C CNN
 F 1 "0.1uF" V 5039 3350 50  0000 C CNN
-F 2 "Capacitor_SMD:C_0805_2012Metric_Pad1.15x1.40mm_HandSolder" H 5238 3200 50  0001 C CNN
+F 2 "Capacitor_SMD:C_0805_2012Metric" H 5238 3200 50  0001 C CNN
 F 3 "~" H 5200 3350 50  0001 C CNN
+F 4 "C49678" H 5200 3350 50  0001 C CNN "LSCS"
 	1    5200 3350
 	0    1    1    0
@@
 AR Path="/60DF69C3/6149FDF7" Ref="#PWR?"  Part="1"
 AR Path="/60DF76F4/6149FDF7" Ref="#PWR?"  Part="1"
-AR Path="/6149EA8A/6149FDF7" Ref="#PWR072"  Part="1"
-F 0 "#PWR072" H 5450 3100 50  0001 C CNN
+AR Path="/6149EA8A/6149FDF7" Ref="#PWR082"  Part="1"
+F 0 "#PWR082" H 5450 3100 50  0001 C CNN
 F 1 "GND" V 5455 3222 50  0000 R CNN
 F 2 "" H 5450 3350 50  0001 C CNN
@@
 AR Path="/60DF69C3/6149FDFE" Ref="#PWR?"  Part="1"
 AR Path="/60DF76F4/6149FDFE" Ref="#PWR?"  Part="1"
-AR Path="/6149EA8A/6149FDFE" Ref="#PWR071"  Part="1"
-F 0 "#PWR071" H 4900 4050 50  0001 C CNN
+AR Path="/6149EA8A/6149FDFE" Ref="#PWR081"  Part="1"
+F 0 "#PWR081" H 4900 4050 50  0001 C CNN
 F 1 "GND" V 4905 4172 50  0000 R CNN
 F 2 "" H 4900 4300 50  0001 C CNN
@@
 PlayerPixels
 $Comp
-L power:+3.3V #PWR0101
+L power:+3.3V #PWR071
 U 1 1 61770704
 P 2500 3250
-F 0 "#PWR0101" H 2500 3100 50  0001 C CNN
+F 0 "#PWR071" H 2500 3100 50  0001 C CNN
 F 1 "+3.3V" H 2515 3423 50  0000 C CNN
 F 2 "" H 2500 3250 50  0001 C CNN
@@
 $EndComp
 $Comp
-L power:+3.3V #PWR0102
+L power:+3.3V #PWR074
 U 1 1 61771465
 P 3300 3250
-F 0 "#PWR0102" H 3300 3100 50  0001 C CNN
+F 0 "#PWR074" H 3300 3100 50  0001 C CNN
 F 1 "+3.3V" H 3315 3423 50  0000 C CNN
 F 2 "" H 3300 3250 50  0001 C CNN
@@
 $EndComp
 $Comp
-L power:+3.3V #PWR0103
+L power:+3.3V #PWR077
 U 1 1 61771C84
 P 4100 3250
-F 0 "#PWR0103" H 4100 3100 50  0001 C CNN
+F 0 "#PWR077" H 4100 3100 50  0001 C CNN
 F 1 "+3.3V" H 4115 3423 50  0000 C CNN
 F 2 "" H 4100 3250 50  0001 C CNN
@@
 $EndComp
 $Comp
-L power:+3.3V #PWR0104
+L power:+3.3V #PWR080
 U 1 1 61772126
 P 4900 3250
-F 0 "#PWR0104" H 4900 3100 50  0001 C CNN
+F 0 "#PWR080" H 4900 3100 50  0001 C CNN
 F 1 "+3.3V" H 4915 3423 50  0000 C CNN
 F 2 "" H 4900 3250 50  0001 C CNN
