File: Power.sch (KiCad schematic (older format))
At the start: 5 parts, among them J2 USB_B_Micro, U2 NCP1117-3.3_SOT223

Commit message: v1.5 Finalized
Parts:
- C12, C13, C14: LSCS (none) -> C15850
- U2: LSCS (none) -> C146799
Changed lines of the file:
@@
 F 2 "Package_TO_SOT_SMD:SOT-223-3_TabPin2" H 5900 3250 50  0001 C CNN
 F 3 "http://www.onsemi.com/pub_link/Collateral/NCP1117-D.PDF" H 6000 2800 50  0001 C CNN
+F 4 "C146799" H 5900 3050 50  0001 C CNN "LSCS"
 	1    5900 3050
 	1    0    0    -1
@@
 F 2 "Capacitor_SMD:C_0805_2012Metric" H 5238 3100 50  0001 C CNN
 F 3 "~" H 5200 3250 50  0001 C CNN
+F 4 "C15850" H 5200 3250 50  0001 C CNN "LSCS"
 	1    5200 3250
 	1    0    0    -1
@@
 F 2 "Capacitor_SMD:C_0805_2012Metric" H 6638 3100 50  0001 C CNN
 F 3 "~" H 6600 3250 50  0001 C CNN
+F 4 "C15850" H 6600 3250 50  0001 C CNN "LSCS"
 	1    6600 3250
 	1    0    0    -1
@@
 F 2 "Capacitor_SMD:C_0805_2012Metric" H 7738 2450 50  0001 C CNN
 F 3 "~" H 7700 2600 50  0001 C CNN
+F 4 "C15850" H 7700 2600 50  0001 C CNN "LSCS"
 	1    7700 2600
 	1    0    0    -1
