File: SingleKey.sch (KiCad schematic (older format))
At the start: 3 parts

Commit message: v1.5 Finalized
Parts:
- U-CAP1: footprint Capacitor_SMD:C_0805_2012Metric_Pad1.15x1.40mm_HandSolder -> Capacitor_SMD:C_0805_2012Metric; LSCS (none) -> C49678
Changed lines of the file:
@@
 $Descr A4 11693 8268
 encoding utf-8
-Sheet 12 19
+Sheet 3 15
 Title ""
 Date ""
@@
 AR Path="/614940F6/61498D85/60A6CE62" Ref="SW-P11"  Part="1"
 AR Path="/614940F6/61498D8D/60A6CE62" Ref="SW-P12"  Part="1"
-F 0 "SW-P10" H 6000 5683 60  0000 C CNN
+F 0 "SW-P1" H 6000 5683 60  0000 C CNN
 F 1 "KEYSW" H 6000 5350 60  0001 C CNN
 F 2 "keyswitches:Kailh_socket_MX" H 6000 5450 60  0001 C CNN
@@
 AR Path="/60DF69C3/60E5DA32" Ref="#PWR?"  Part="1"
 AR Path="/60DF76F4/60E5DA32" Ref="#PWR?"  Part="1"
-AR Path="/614940F6/61498D3D/60E5DA32" Ref="#PWR016"  Part="1"
-AR Path="/614940F6/61498D42/60E5DA32" Ref="#PWR020"  Part="1"
-AR Path="/614940F6/61498D47/60E5DA32" Ref="#PWR024"  Part="1"
-AR Path="/614940F6/61498D4F/60E5DA32" Ref="#PWR028"  Part="1"
-AR Path="/614940F6/61498D58/60E5DA32" Ref="#PWR032"  Part="1"
-AR Path="/614940F6/61498D60/60E5DA32" Ref="#PWR036"  Part="1"
-AR Path="/614940F6/61498D68/60E5DA32" Ref="#PWR040"  Part="1"
-AR Path="/614940F6/61498D70/60E5DA32" Ref="#PWR044"  Part="1"
-AR Path="/614940F6/61498D77/60E5DA32" Ref="#PWR048"  Part="1"
-AR Path="/614940F6/61498D7E/60E5DA32" Ref="#PWR052"  Part="1"
-AR Path="/614940F6/61498D85/60E5DA32" Ref="#PWR056"  Part="1"
-AR Path="/614940F6/61498D8D/60E5DA32" Ref="#PWR060"  Part="1"
-F 0 "#PWR060" H 6400 5200 50  0001 C CNN
+AR Path="/614940F6/61498D3D/60E5DA32" Ref="#PWR026"  Part="1"
+AR Path="/614940F6/61498D42/60E5DA32" Ref="#PWR030"  Part="1"
+AR Path="/614940F6/61498D47/60E5DA32" Ref="#PWR034"  Part="1"
+AR Path="/614940F6/61498D4F/60E5DA32" Ref="#PWR038"  Part="1"
+AR Path="/614940F6/61498D58/60E5DA32" Ref="#PWR042"  Part="1"
+AR Path="/614940F6/61498D60/60E5DA32" Ref="#PWR046"  Part="1"
+AR Path="/614940F6/61498D68/60E5DA32" Ref="#PWR050"  Part="1"
+AR Path="/614940F6/61498D70/60E5DA32" Ref="#PWR054"  Part="1"
+AR Path="/614940F6/61498D77/60E5DA32" Ref="#PWR058"  Part="1"
+AR Path="/614940F6/61498D7E/60E5DA32" Ref="#PWR062"  Part="1"
+AR Path="/614940F6/61498D85/60E5DA32" Ref="#PWR066"  Part="1"
+AR Path="/614940F6/61498D8D/60E5DA32" Ref="#PWR070"  Part="1"
+F 0 "#PWR070" H 6400 5200 50  0001 C CNN
 F 1 "GND" V 6405 5322 50  0000 R CNN
 F 2 "" H 6400 5450 50  0001 C CNN
@@
 AR Path="/614940F6/61498D85/60BFC128" Ref="U-CAP11"  Part="1"
 AR Path="/614940F6/61498D8D/60BFC128" Ref="U-CAP12"  Part="1"
-F 0 "U-CAP10" V 3700 3750 50  0000 C CNN
+F 0 "U-CAP1" V 3700 3750 50  0000 C CNN
 F 1 "0.1uF" V 3789 3600 50  0000 C CNN
-F 2 "Capacitor_SMD:C_0805_2012Metric_Pad1.15x1.40mm_HandSolder" H 3988 3450 50  0001 C CNN
+F 2 "Capacitor_SMD:C_0805_2012Metric" H 3988 3450 50  0001 C CNN
 F 3 "~" H 3950 3600 50  0001 C CNN
+F 4 "C49678" H 3950 3600 50  0001 C CNN "LSCS"
 	1    3950 3600
 	0    1    1    0
@@
 AR Path="/614940F6/61498D85/60BFC130" Ref="U-RGB11"  Part="1"
 AR Path="/614940F6/61498D8D/60BFC130" Ref="U-RGB12"  Part="1"
-F 0 "U-RGB10" H 3500 4200 50  0000 L CNN
+F 0 "U-RGB1" H 3500 4200 50  0000 L CNN
 F 1 "Reverse Mounted NeoPixel" H 3150 5100 50  0000 L CNN
 F 2 "Keebio-Parts:SK6812-MINI-E" H 3700 3800 50  0001 L TNN
@@
 AR Path="/60DF69C3/60BFC13F" Ref="#PWR?"  Part="1"
 AR Path="/60DF76F4/60BFC13F" Ref="#PWR?"  Part="1"
-AR Path="/614940F6/61498D3D/60BFC13F" Ref="#PWR015"  Part="1"
-AR Path="/614940F6/61498D42/60BFC13F" Ref="#PWR019"  Part="1"
-AR Path="/614940F6/61498D47/60BFC13F" Ref="#PWR023"  Part="1"
-AR Path="/614940F6/61498D4F/60BFC13F" Ref="#PWR027"  Part="1"
-AR Path="/614940F6/61498D58/60BFC13F" Ref="#PWR031"  Part="1"
-AR Path="/614940F6/61498D60/60BFC13F" Ref="#PWR035"  Part="1"
-AR Path="/614940F6/61498D68/60BFC13F" Ref="#PWR039"  Part="1"
-AR Path="/614940F6/61498D70/60BFC13F" Ref="#PWR043"  Part="1"
-AR Path="/614940F6/61498D77/60BFC13F" Ref="#PWR047"  Part="1"
-AR Path="/614940F6/61498D7E/60BFC13F" Ref="#PWR051"  Part="1"
-AR Path="/614940F6/61498D85/60BFC13F" Ref="#PWR055"  Part="1"
-AR Path="/614940F6/61498D8D/60BFC13F" Ref="#PWR059"  Part="1"
-F 0 "#PWR059" H 4200 3350 50  0001 C CNN
+AR Path="/614940F6/61498D3D/60BFC13F" Ref="#PWR025"  Part="1"
+AR Path="/614940F6/61498D42/60BFC13F" Ref="#PWR029"  Part="1"
+AR Path="/614940F6/61498D47/60BFC13F" Ref="#PWR033"  Part="1"
+AR Path="/614940F6/61498D4F/60BFC13F" Ref="#PWR037"  Part="1"
+AR Path="/614940F6/61498D58/60BFC13F" Ref="#PWR041"  Part="1"
+AR Path="/614940F6/61498D60/60BFC13F" Ref="#PWR045"  Part="1"
+AR Path="/614940F6/61498D68/60BFC13F" Ref="#PWR049"  Part="1"
+AR Path="/614940F6/61498D70/60BFC13F" Ref="#PWR053"  Part="1"
+AR Path="/614940F6/61498D77/60BFC13F" Ref="#PWR057"  Part="1"
+AR Path="/614940F6/61498D7E/60BFC13F" Ref="#PWR061"  Part="1"
+AR Path="/614940F6/61498D85/60BFC13F" Ref="#PWR065"  Part="1"
+AR Path="/614940F6/61498D8D/60BFC13F" Ref="#PWR069"  Part="1"
+F 0 "#PWR069" H 4200 3350 50  0001 C CNN
 F 1 "GND" V 4205 3472 50  0000 R CNN
 F 2 "" H 4200 3600 50  0001 C CNN
@@
 AR Path="/60DF69C3/60BFC146" Ref="#PWR?"  Part="1"
 AR Path="/60DF76F4/60BFC146" Ref="#PWR?"  Part="1"
-AR Path="/614940F6/61498D3D/60BFC146" Ref="#PWR014"  Part="1"
-AR Path="/614940F6/61498D42/60BFC146" Ref="#PWR018"  Part="1"
-AR Path="/614940F6/61498D47/60BFC146" Ref="#PWR022"  Part="1"
-AR Path="/614940F6/61498D4F/60BFC146" Ref="#PWR026"  Part="1"
-AR Path="/614940F6/61498D58/60BFC146" Ref="#PWR030"  Part="1"
-AR Path="/614940F6/61498D60/60BFC146" Ref="#PWR034"  Part="1"
-AR Path="/614940F6/61498D68/60BFC146" Ref="#PWR038"  Part="1"
-AR Path="/614940F6/61498D70/60BFC146" Ref="#PWR042"  Part="1"
-AR Path="/614940F6/61498D77/60BFC146" Ref="#PWR046"  Part="1"
-AR Path="/614940F6/61498D7E/60BFC146" Ref="#PWR050"  Part="1"
-AR Path="/614940F6/61498D85/60BFC146" Ref="#PWR054"  Part="1"
-AR Path="/614940F6/61498D8D/60BFC146" Ref="#PWR058"  Part="1"
-F 0 "#PWR058" H 3650 4300 50  0001 C CNN
+AR Path="/614940F6/61498D3D/60BFC146" Ref="#PWR024"  Part="1"
+AR Path="/614940F6/61498D42/60BFC146" Ref="#PWR028"  Part="1"
+AR Path="/614940F6/61498D47/60BFC146" Ref="#PWR032"  Part="1"
+AR Path="/614940F6/61498D4F/60BFC146" Ref="#PWR036"  Part="1"
+AR Path="/614940F6/61498D58/60BFC146" Ref="#PWR040"  Part="1"
+AR Path="/614940F6/61498D60/60BFC146" Ref="#PWR044"  Part="1"
+AR Path="/614940F6/61498D68/60BFC146" Ref="#PWR048"  Part="1"
+AR Path="/614940F6/61498D70/60BFC146" Ref="#PWR052"  Part="1"
+AR Path="/614940F6/61498D77/60BFC146" Ref="#PWR056"  Part="1"
+AR Path="/614940F6/61498D7E/60BFC146" Ref="#PWR060"  Part="1"
+AR Path="/614940F6/61498D85/60BFC146" Ref="#PWR064"  Part="1"
+AR Path="/614940F6/61498D8D/60BFC146" Ref="#PWR068"  Part="1"
+F 0 "#PWR068" H 3650 4300 50  0001 C CNN
 F 1 "GND" V 3655 4422 50  0000 R CNN
 F 2 "" H 3650 4550 50  0001 C CNN
@@
 AR Path="/60DF69C3/612471BD" Ref="#PWR?"  Part="1"
 AR Path="/60DF76F4/612471BD" Ref="#PWR?"  Part="1"
-AR Path="/614940F6/61498D3D/612471BD" Ref="#PWR013"  Part="1"
-AR Path="/614940F6/61498D42/612471BD" Ref="#PWR017"  Part="1"
-AR Path="/614940F6/61498D47/612471BD" Ref="#PWR021"  Part="1"
-AR Path="/614940F6/61498D4F/612471BD" Ref="#PWR025"  Part="1"
-AR Path="/614940F6/61498D58/612471BD" Ref="#PWR029"  Part="1"
-AR Path="/614940F6/61498D60/612471BD" Ref="#PWR033"  Part="1"
-AR Path="/614940F6/61498D68/612471BD" Ref="#PWR037"  Part="1"
-AR Path="/614940F6/61498D70/612471BD" Ref="#PWR041"  Part="1"
-AR Path="/614940F6/61498D77/612471BD" Ref="#PWR045"  Part="1"
-AR Path="/614940F6/61498D7E/612471BD" Ref="#PWR049"  Part="1"
-AR Path="/614940F6/61498D85/612471BD" Ref="#PWR053"  Part="1"
-AR Path="/614940F6/61498D8D/612471BD" Ref="#PWR057"  Part="1"
-F 0 "#PWR057" H 3650 3350 50  0001 C CNN
+AR Path="/614940F6/61498D3D/612471BD" Ref="#PWR023"  Part="1"
+AR Path="/614940F6/61498D42/612471BD" Ref="#PWR027"  Part="1"
+AR Path="/614940F6/61498D47/612471BD" Ref="#PWR031"  Part="1"
+AR Path="/614940F6/61498D4F/612471BD" Ref="#PWR035"  Part="1"
+AR Path="/614940F6/61498D58/612471BD" Ref="#PWR039"  Part="1"
+AR Path="/614940F6/61498D60/612471BD" Ref="#PWR043"  Part="1"
+AR Path="/614940F6/61498D68/612471BD" Ref="#PWR047"  Part="1"
+AR Path="/614940F6/61498D70/612471BD" Ref="#PWR051"  Part="1"
+AR Path="/614940F6/61498D77/612471BD" Ref="#PWR055"  Part="1"
+AR Path="/614940F6/61498D7E/612471BD" Ref="#PWR059"  Part="1"
+AR Path="/614940F6/61498D85/612471BD" Ref="#PWR063"  Part="1"
+AR Path="/614940F6/61498D8D/612471BD" Ref="#PWR067"  Part="1"
+F 0 "#PWR067" H 3650 3350 50  0001 C CNN
 F 1 "+3.3V" H 3665 3673 50  0000 C CNN
 F 2 "" H 3650 3500 50  0001 C CNN
