File: OSFRD.kicad_pcb (KiCad board)
At the start: 2 copper layers, 186 x 99.1 mm, 89 parts, among them J1 20 Pin, J2 USB_B_Micro, J3 STEMMA QT, J4 Debug, SW1 SW_PUSH, SW2 SW_PUSH, SW3 SW_PUSH, SW4 SW_PUSH, SW5 SW_PUSH, SW6 SW_PUSH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

Commit message: v1.5 Finalized
Parts:
- removed C1, C10, C11, C17, C2, C4, C6, C7, C8, C9: 100n, Capacitor_SMD:C_0402_1005Metric
- removed C12, C13, C14: 10u, Capacitor_SMD:C_0805_2012Metric
- removed C15, C16: 27p, Capacitor_SMD:C_0402_1005Metric
- removed C3, C5: 1u, Capacitor_SMD:C_0402_1005Metric
- removed J1: 20 Pin, Connector_PinSocket_2.54mm:PinSocket_2x10_P2.54mm_Vertical
- removed J2: USB_B_Micro, RP2040_minimal:USB_Micro-B_Amphenol_10103594-0001LF_Horizontal_modified
- removed J4: Debug, Connector_PinSocket_2.54mm:PinSocket_1x03_P2.54mm_Vertical
- removed R1, R2: 27, Capacitor_SMD:C_0402_1005Metric
- removed the R3 at (181.1, 78.8)
- removed R4: 1k, Capacitor_SMD:C_0402_1005Metric
- removed R5: DNF, Capacitor_SMD:C_0402_1005Metric
- removed the REF** at (144.0, 73.5)
- removed the REF** at (144.0, 128.1)
- removed the REF** at (144.0, 37.0)
- removed the REF** at (236.0, 37.0)
- removed SW3: SW_PUSH, Button_Switch_THT:SW_Tactile_SPST_Angled_PTS645Vx83-2LFS
- removed SW8: SW_Push, Button_Switch_SMD:SW_Push_1P1T_NO_CK_KSC7xxJ
- removed U2: NCP1117-3.3_SOT223, Package_TO_SOT_SMD:SOT-223-3_TabPin2
- removed U3: W25Q128JVS, Package_SO:SOIC-8_5.23x5.23mm_P1.27mm
- removed Y1: ABLS-12.000MHZ-B4-T, RP2040_minimal:Crystal_SMD_HC49-US
- added BROOK: 20 Pin, Connector_PinSocket_2.54mm:PinSocket_2x10_P2.54mm_Vertical_SMD, B.Cu at (215.7, 92.2)
- added G***: LOGO, OSFRD:sleepunit, F.Cu at (233.6, 116.4)
- added REF**: Shinoo_M3_Standoff, BarketImages:Shinoo_M3_Standoff, F.Cu at (159.0, 73.5)
- added REF**: Shinoo_M3_Standoff, BarketImages:Shinoo_M3_Standoff, F.Cu at (159.0, 128.1)
- added REF**: Shinoo_M3_Standoff, BarketImages:Shinoo_M3_Standoff, F.Cu at (159.0, 37.0)
- added REF**: Shinoo_M3_Standoff, BarketImages:Shinoo_M3_Standoff, F.Cu at (251.0, 37.0)
- added SETTINGS: SW_PUSH, Button_Switch_THT:SW_Tactile_SPST_Angled_PTS645Vx83-2LFS, F.Cu at (224.2, 35.9)
- STEMMA QT: renamed from J3; moved to B.Cu
- U-CAP1, U-CAP10, U-CAP11, U-CAP12, U-CAP13, U-CAP14, U-CAP15, U-CAP16, U-CAP2, U-CAP3, U-CAP4, U-CAP5, U-CAP6, U-CAP7, U-CAP8, U-CAP9: footprint Capacitor_SMD:C_0805_2012Metric_Pad1.15x1.40mm_HandSolder -> Capacitor_SMD:C_0805_2012Metric
- U1: value RP2040 -> Pico; footprint RP2040_minimal:RP2040-QFN-56 -> MCU_RaspberryPi_and_Boards:RPi_Pico_SMD_TH
- moved U1 111.7 mm to (80.0, 100.0), turned to 270 degrees
- moved STEMMA QT 44.7 mm to (86.3, 50.0)
- moved REF** 15.0 mm to (251.0, 128.1)
- moved SW-P10 12.0 mm to (182.7, 72.4)
- moved SW-P11 12.0 mm to (211.5, 72.4)
- moved SW-P12 12.0 mm to (240.3, 79.5)
- moved SW-P5 12.0 mm to (158.3, 57.2)
- moved SW-P6 12.0 mm to (182.7, 41.2)
- moved SW-P7 12.0 mm to (211.5, 41.1)
- moved SW-P8 12.0 mm to (239.9, 48.3)
- moved SW-P9 12.0 mm to (158.3, 88.4)
- moved U-CAP10 12.0 mm to (177.7, 76.9)
- moved U-CAP11 12.0 mm to (206.5, 76.9)
- moved U-CAP12 12.0 mm to (235.3, 84.0)
- moved U-CAP5 12.0 mm to (153.3, 61.7)
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- renumbered SW6 to HOME, SW5 to L3, SW7 to R3, SW4 to SELECT, SW1 to START, SW2 to TOUCH
Connections:
- HOME pad 1: /GPIO23 -> /GPIO4
- SELECT pad 1: /GPIO24 -> /GPIO3
- START pad 1: /GPIO25 -> /GPIO0
- SW-P1 pad 2: /GPIO16 -> /GPIO20
- SW-P11 pad 2: /GPIO14 -> /GPIO16
- SW-P12 pad 2: /GPIO13 -> /GPIO19
- SW-P2 pad 2: /GPIO20 -> /GPIO8
- SW-P3 pad 2: /GPIO19 -> /GPIO1
- SW-P4 pad 2: /GPIO21 -> /GPIO14
- SW-P5 pad 2: /GPIO28_ADC2 -> /GPIO13
- SW-P6 pad 2: /GPIO29_ADC3 -> /GPIO9
- SW-P7 pad 2: /GPIO0 -> /GPIO10
- SW-P8 pad 2: /GPIO3 -> /GPIO12
- U-RGB3 pad 2: /GPIO22 -> /GPIO2
- U1 pad 1: +3V3 -> /GPIO0
- U1 pad 10: +3V3 -> /GPIO7
- U1 pad 11: /MCU/GPIO8 -> /GPIO8
- U1 pad 12: /MCU/GPIO9 -> /GPIO9
- U1 pad 13: /MCU/GPIO10 -> GND
- U1 pad 14: /MCU/GPIO11 -> /GPIO10
- U1 pad 15: /MCU/GPIO12 -> /GPIO11
- U1 pad 16: /GPIO13 -> /GPIO12
- U1 pad 17: /GPIO14 -> /GPIO13
- U1 pad 18: /MCU/GPIO15 -> GND
- U1 pad 19: GND -> /GPIO14
- U1 pad 2: /GPIO0 -> /GPIO1
- U1 pad 20: /MCU/XIN -> Net-(U1-Pad20)
- U1 pad 21: /MCU/XOUT -> /GPIO16
- U1 pad 22: +3V3 -> /GPIO17
- U1 pad 23: +1V1 -> GND
- U1 pad 24: /MCU/SWCLK -> /GPIO18
- U1 pad 25: /MCU/SWDIO -> /GPIO19
- U1 pad 26: Net-(U1-Pad26) -> /GPIO20
- U1 pad 27: /GPIO16 -> Net-(U1-Pad27)
- U1 pad 28: /GPIO17 -> GND
- U1 pad 29: /GPIO18 -> Net-(U1-Pad29)
- U1 pad 3: /GPIO1 -> GND
- U1 pad 30: /GPIO19 -> Net-(U1-Pad30)
- U1 pad 31: /GPIO20 -> /GPIO26_I2C1_SDA
- U1 pad 32: /GPIO21 -> /GPIO27_I2C1_SCL
- U1 pad 33: +3V3 -> GND
- U1 pad 34: /GPIO22 -> Net-(U1-Pad34)
- U1 pad 35: /GPIO23 -> Net-(U1-Pad35)
- U1 pad 36: /GPIO24 -> +3V3
- U1 pad 37: /GPIO25 -> Net-(U1-Pad37)
- U1 pad 38: /GPIO26_I2C1_SDA -> GND
- U1 pad 39: /GPIO27_I2C1_SCL -> +5V
- U1 pad 4: /MCU/GPIO2 -> /GPIO2
- U1 pad 40: /GPIO28_ADC2 -> Net-(U1-Pad40)
- U1 pad 41: /GPIO29_ADC3 -> Net-(U1-Pad41)
- U1 pad 42: +3V3 -> Net-(U1-Pad42)
- U1 pad 43: +3V3 -> Net-(U1-Pad43)
- U1 pad 6: /MCU/GPIO4 -> /GPIO4
- U1 pad 8: /GPIO6 -> GND
- U1 pad 9: /GPIO7 -> /GPIO6
Routing:
- net /GPIO24: track 225.8 -> 0.00 mm, vias 6 -> 0
- net /GPIO4: track 0.00 -> 224.5 mm, vias 0 -> 6
- net /GPIO25: track 221.2 -> 0.00 mm, vias 5 -> 0
- net /GPIO9: track 0.00 -> 213.3 mm, vias 0 -> 2
- net /GPIO23: track 210.0 -> 0.00 mm, vias 5 -> 0
- net /GPIO10: track 0.00 -> 207.8 mm, vias 0 -> 2
- net /GPIO12: track 0.00 -> 202.7 mm, vias 0 -> 2
- net /GPIO8: track 0.00 -> 194.7 mm, vias 0 -> 3
- net /GPIO1: track 38.6 -> 212.2 mm, vias 4 -> 1
- net /GPIO21: track 163.3 -> 0.00 mm, vias 4 -> 0
- net /GPIO11: track 0.00 -> 159.1 mm
- net /GPIO28_ADC2: track 148.1 -> 0.00 mm, vias 7 -> 0
- net /GPIO22: track 143.0 -> 0.00 mm, vias 2 -> 0
- net /GPIO0: track 123.5 -> 260.3 mm, vias 6 -> 4
- net /GPIO29_ADC3: track 127.4 -> 0.00 mm, vias 5 -> 0
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Other:
- board size 186 x 99.1 mm -> 201 x 99.1 mm
- net class Default: trace_width 0.25 -> 0.2
